File: hardware/finishBoard/FinishControllerBoard_v1.kicad_pcb (KiCad board)
At the start: 2 copper layers, 106 parts, among them J1 Conn_01x04, J10 Comm, J11 Conn_01x02, J2 LCD_Top_Half, J3 LCD_Bottom_Half, J4 Time2, J5 Time1, J6 React1, J7 React2, J8 Analog, J9 Digital, U1 74HC595, U11 7414, U12 74HC137, U14 7414, U15 7414, U16 74HC137, U17 74HC137, U2 7414, U3 74HC595, U4 L78L05_SOT89, U5 7414, U7 7414, U8 74HC137, U9 7414

Commit message: Finish Control Board completion for order
Parts:
- removed C16, C17, C18, C19, C7, C8: 0.1uF, Capacitor_SMD:C_0805_2012Metric
- removed D18, D19, D20, D21, D22, D23, D24, D25, D26, D27, D28, D29, D30, D31, D32, D33, D34: 1N4148W, Diode_SMD:D_SOD-123
- removed D45, D46: Green, LED_SMD:LED_0805_2012Metric
- removed J10: Comm, Connector_JST:JST_EH_B3B-EH-A_1x03_P2.50mm_Vertical
- removed J11: Conn_01x02, Connector_JST:JST_XH_B2B-XH-A_1x02_P2.50mm_Vertical
- removed J7: React2, Connector_JST:JST_VH_B10P-VH-B_1x10_P3.96mm_Vertical
- removed U11, U14, U15, U9: 7414, Package_SO:SOIC-14_3.9x8.7mm_P1.27mm
- removed U12, U16, U17, U8: 74HC137, Package_SO:SOIC-16_3.9x9.9mm_P1.27mm
- added C13: 0.1uF, Capacitor_SMD:C_0805_2012Metric, F.Cu at (213.2, 28.5)
- added Q1: BSS138, Package_TO_SOT_SMD:SOT-23_Handsoldering, F.Cu at (195.2, -0.79)
- added Q2: BSS138, Package_TO_SOT_SMD:SOT-23_Handsoldering, F.Cu at (189.7, 4.79)
- added R11: 10k, Resistor_SMD:R_0805_2012Metric, F.Cu at (191.4, -0.85)
- added R14: 10k, Resistor_SMD:R_0805_2012Metric, F.Cu at (193.5, 2.80)
- added R15: 10k, Resistor_SMD:R_0805_2012Metric, F.Cu at (190.7, 1.90)
- added R16: 10k, Resistor_SMD:R_0805_2012Metric, F.Cu at (196.3, 2.10)
- added R17: 150, Resistor_SMD:R_0805_2012Metric, F.Cu at (188.6, -1.55)
- added R20: 0, Resistor_SMD:R_0805_2012Metric, F.Cu at (187.9, 1.20)
- added R21: 0, Resistor_SMD:R_0805_2012Metric, F.Cu at (194.2, 5.60)
- added R22: 0, Resistor_SMD:R_0805_2012Metric, F.Cu at (197.0, 4.85)
- added R23: 100, Resistor_SMD:R_0805_2012Metric, F.Cu at (209.1, 14.4)
- added R24: 100, Resistor_SMD:R_0805_2012Metric, F.Cu at (206.5, 14.4)
- added R25: 100, Resistor_SMD:R_0805_2012Metric, F.Cu at (204.0, 14.4)
- added R26: 100, Resistor_SMD:R_0805_2012Metric, F.Cu at (201.5, 14.4)
- added R27: 560, Resistor_SMD:R_0805_2012Metric, F.Cu at (209.0, -13.4)
- added R28: 10k, Resistor_SMD:R_0805_2012Metric, F.Cu at (184.5, -16.0)
- C5: value 10nF -> 10uF
- D15, D16, D17: value 1N4148W -> Green; footprint Diode_SMD:D_SOD-123 -> LED_SMD:LED_0805_2012Metric_Pad1.15x1.40mm_HandSolder
- H1, H2, H3, H4: footprint MountingHole:MountingHole_3.2mm_M3_Pad_TopBottom -> MountingHole:MountingHole_2.5mm_Pad
- J1: value Conn_01x04 -> Sensors
- J2: value LCD_Top_Half -> Comm; footprint Connector_JST:JST_VH_B8P-VH-B_1x08_P3.96mm_Vertical -> Connector_JST:JST_EH_B3B-EH-A_1x03_P2.50mm_Vertical
- J3: value LCD_Bottom_Half -> 12V Pwr; footprint Connector_JST:JST_VH_B8P-VH-B_1x08_P3.96mm_Vertical -> Connector_Molex:Molex_Nano-Fit_105309-xx02_1x02_P2.50mm_Vertical
- J4, J5: footprint Connector_JST:JST_VH_B10P-VH-B_1x10_P3.96mm_Vertical -> Connector_JST:JST_EH_B10B-EH-A_1x10_P2.50mm_Vertical
- J6: value React1 -> Dsply Pwr; footprint Connector_JST:JST_VH_B10P-VH-B_1x10_P3.96mm_Vertical -> Connector_Molex:Molex_Nano-Fit_105309-xx04_1x04_P2.50mm_Vertical
- R10: value 200 -> 560
- R5: value 22 -> 100
- R6: value 12k -> 100
- R7: value 1k -> 100
- U1: value 74HC595 -> 74HCT238
- U2: value 7414 -> 74HCT238; footprint Package_SO:SOIC-14_3.9x8.7mm_P1.27mm -> Package_SO:SOIC-16_3.9x9.9mm_P1.27mm
- U3: value 74HC595 -> 74LVC2G14; footprint Package_SO:SOIC-16_3.9x9.9mm_P1.27mm -> Package_TO_SOT_SMD:SOT-23-6_Handsoldering
- U4: value L78L05_SOT89 -> L78M05CDT; footprint Package_TO_SOT_SMD:SOT-89-3 -> PCM_Package_TO_SOT_SMD_AKL:TO-252-2
- U5: value 7414 -> 74HCT244; footprint Package_SO:SOIC-14_3.9x8.7mm_P1.27mm -> Package_SO:SOIC-20W_7.5x12.8mm_P1.27mm
- U7: value 7414 -> AP2112K-3.3; footprint Package_SO:SOIC-14_3.9x8.7mm_P1.27mm -> Package_TO_SOT_SMD:SOT-23-5_HandSoldering
- moved D38 333.3 mm to (222.8, 27.6)
- moved D37 327.4 mm to (217.9, 27.6)
- moved D42 325.4 mm to (222.8, 30.1)
- moved J4 322.7 mm to (227.7, 42.8), turned to 90 degrees
- moved D41 319.5 mm to (217.9, 30.1)
- moved D17 314.8 mm to (197.0, -29.0), turned to 180 degrees
- moved D6 314.5 mm to (222.8, 20.1)
- moved D9 314.1 mm to (217.9, 22.6)
- moved D14 312.1 mm to (222.8, 25.1)
- moved D15 310.9 mm to (208.0, -16.2)
- moved D5 308.6 mm to (217.9, 20.1)
- moved C4 308.5 mm to (222.5, -13.0), turned to 180 degrees
- moved D10 306.5 mm to (222.8, 22.6)
- moved D13 306.1 mm to (217.9, 25.1)
- moved D39 305.8 mm to (194.0, 35.5), turned to 180 degrees
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Connections:
- C3 pad 1: GND -> +5V
- C3 pad 2: +5V -> GND
- C4 pad 2: +5V -> +3.3V
- C5 pad 1: +5V -> +3.3V
- C6 pad 1: +5V -> +3.3V
- D10 pad 1: /Digit Demux Right/Time2_Thousandths -> /Time2_Hundredths
- D11 pad 1: /Digit Demux Right/Time2_Hundredths -> +5V
- D11 pad 2: GND -> /Time1_Hundredths
- D12 pad 1: /Digit Demux Right/Time2_Tenths -> /Time1_Hundredths
- D13 pad 1: /Digit Demux Right/Time2_Ones -> +5V
- D13 pad 2: GND -> /Time2_Tenths
- D14 pad 1: /Digit Demux Right/Time2_Tens -> /Time2_Tenths
- D15 pad 1: +5V -> GND
- D15 pad 2: /React2_Thousandths -> Net-(D15-A)
- D16 pad 1: +5V -> GND
- D16 pad 2: /React2_Hundredths -> Net-(D16-A)
- D17 pad 1: +5V -> GND
- D17 pad 2: /React2_Tenths -> Net-(D17-A)
- D35 pad 2: /LCD Left Latching/React1_Thousandths -> /Time1_Tenths
- D36 pad 1: +5V -> /Time1_Tenths
- D36 pad 2: /LCD Left Latching/React1_Hundredths -> GND
- D37 pad 2: /LCD Left Latching/React1_Tenths -> /Time2_Ones
- D38 pad 1: +5V -> /Time2_Ones
- D38 pad 2: /LCD Left Latching/React1_Ones -> GND
- D39 pad 2: /LCD Left Latching/React1_Tens -> /Time1_Ones
- D40 pad 1: /LCD Left Latching/React1_Thousandths -> /Time1_Ones
- D41 pad 1: /LCD Left Latching/React1_Hundredths -> +5V
- D41 pad 2: GND -> /Time2_Tens
- D42 pad 1: /LCD Left Latching/React1_Tenths -> /Time2_Tens
- D43 pad 1: /LCD Left Latching/React1_Ones -> +5V
- D43 pad 2: GND -> /Time1_Tens
- D44 pad 1: /LCD Left Latching/React1_Tens -> /Time1_Tens
- D5 pad 2: /Digit Demux Right/Time2_Thousandths -> /Time2_Thousandths
- D6 pad 1: +5V -> /Time2_Thousandths
- D6 pad 2: /Digit Demux Right/Time2_Hundredths -> GND
- D7 pad 2: /Digit Demux Right/Time2_Tenths -> /Time1_Thousandths
- D8 pad 1: +5V -> /Time1_Thousandths
- D8 pad 2: /Digit Demux Right/Time2_Ones -> GND
- D9 pad 2: /Digit Demux Right/Time2_Tens -> /Time2_Hundredths
- J2 pad 1: GND -> /Logic Level Shifter/Tx_HV_In
- J2 pad 2: +5V -> /Logic Level Shifter/Rx_HV_Out
- J2 pad 3: Net-(J2-Pin_3) -> GND
- J3 pad 1: unconnected-(J3-Pin_1-Pad1) -> +12V
- J3 pad 2: unconnected-(J3-Pin_2-Pad2) -> GND
- J4 pad 10: /Digit Demux Right/Time2_Thousandths -> /Time2_Thousandths
- J4 pad 5: Time2_Decimal_Point -> Decimal_Point
- J4 pad 6: /Digit Demux Right/Time2_Tens -> /Time2_Tens
- J4 pad 7: /Digit Demux Right/Time2_Ones -> /Time2_Ones
- J4 pad 8: /Digit Demux Right/Time2_Tenths -> /Time2_Tenths
- J4 pad 9: /Digit Demux Right/Time2_Hundredths -> /Time2_Hundredths
- J5 pad 5: Time1_Decimal_Point -> Decimal_Point
- J6 pad 1: AD0 -> +12V
- J6 pad 2: AD3 -> GND
- J6 pad 3: AD1 -> GND
- J6 pad 4: AD2 -> +5V
- J8 pad 10: Clock2 -> /A6
- J8 pad 11: Latch2 -> /A7
- J8 pad 9: Ser2 -> /A5/SCL
- J9 pad 7: Ser1 -> /*D6
- J9 pad 8: Clock1 -> /*D5
- J9 pad 9: Latch1 -> /D4
- R10 pad 1: Net-(D46-A) -> Net-(D16-A)
- R10 pad 2: +5V -> +3.3V
- R18 pad 1: LCD_R/NW -> Net-(U5-2A1)
- R18 pad 2: /D8 -> /D7
- R19 pad 1: LCD_E -> Net-(U5-2A0)
- R19 pad 2: /*D9 -> /*D6
- R5 pad 1: Net-(J3-Pin_7) -> /A2
- R5 pad 2: +5V -> BCD_Lane1
- R6 pad 1: Net-(J2-Pin_3) -> /A3
- R6 pad 2: +5V -> BCD_Lane2
- R7 pad 1: GND -> Net-(U5-2A3)
- R7 pad 2: Net-(J2-Pin_3) -> /*D9
- R8 pad 1: /D7 -> Net-(U5-2A2)
- R8 pad 2: LCD_RS/CS -> /D8
- R9 pad 1: Net-(D45-A) -> Net-(D17-A)
- U1 pad 1: Time2_Decimal_Point -> BCD_MuxA
- U1 pad 10: +5V -> unconnected-(U1-Y5-Pad10)
- U1 pad 11: Clock2 -> /Time1_Tens
- U1 pad 12: Latch2 -> /Time1_Ones
- U1 pad 13: GND -> /Time1_Tenths
- U1 pad 14: Ser2 -> /Time1_Hundredths
- U1 pad 15: Time1_Decimal_Point -> /Time1_Thousandths
- U1 pad 2: React1_Decimal_Point -> BCD_MuxB
- U1 pad 3: React2_Decimal_Point -> BCD_MuxC
- U1 pad 4: AD0 -> GND
- U1 pad 5: AD1 -> BCD_Lane1
- U1 pad 6: AD2 -> +5V
- U1 pad 7: AD3 -> unconnected-(U1-Y7-Pad7)
- U2 pad 1: Net-(C1-Pad1) -> BCD_MuxA
- U2 pad 11: GND -> /Time2_Tens
- U2 pad 12: unconnected-(U2-Pad12) -> /Time2_Ones
- U2 pad 13: GND -> /Time2_Tenths
- U2 pad 14: +5V -> /Time2_Hundredths
- U2 pad 2: /FinishSensors/Lane1_FinishLine -> BCD_MuxB
- U2 pad 3: Net-(C2-Pad1) -> BCD_MuxC
- U2 pad 4: /FinishSensors/Lane2_FinishLine -> GND
- U2 pad 5: BCD_Time -> BCD_Lane2
- U2 pad 6: BCD_React -> +5V
- U2 pad 7: GND -> unconnected-(U2-Y7-Pad7)
- U2 pad 8: BCD_Lane2 -> GND
- U2 pad 9: BCD_Lane1 -> unconnected-(U2-Y6-Pad9)
- U3 pad 1: BCD_MuxB -> Net-(C1-Pad1)
- U3 pad 2: BCD_MuxC -> GND
- U3 pad 3: BCD_Time -> Net-(C2-Pad1)
- U3 pad 4: BCD_Lane1 -> /FinishSensors/Lane2_FinishLine
- U3 pad 5: unconnected-(U3-QF-Pad5) -> +3.3V
- U3 pad 6: unconnected-(U3-QG-Pad6) -> /FinishSensors/Lane1_FinishLine
- U4 pad 1: +5V -> +12V
- U4 pad 3: +12V -> +5V
- U5 pad 10: /Digit Demux Right/Time2_Hundredths -> GND
- U5 pad 11: Net-(U16-~{Y1}) -> Net-(U5-2A3)
- U5 pad 12: /Digit Demux Right/Time2_Thousandths -> AD0
- U5 pad 13: Net-(U16-~{Y0}) -> Net-(U5-2A2)
- U5 pad 14: +5V -> BCD_MuxC
- U5 pad 2: unconnected-(U5-Pad2) -> Net-(U5-1A0)
- U5 pad 3: Net-(U16-~{Y2}) -> AD1
- U5 pad 4: /Digit Demux Right/Time2_Tenths -> Net-(U5-1A1)
- U5 pad 5: Net-(U16-~{Y3}) -> AD2
- U5 pad 6: /Digit Demux Right/Time2_Ones -> Net-(U5-1A2)
- U5 pad 7: GND -> AD3
- U5 pad 8: /Digit Demux Right/Time2_Tens -> Net-(U5-1A3)
- U5 pad 9: Net-(U16-~{Y4}) -> Decimal_Point
- U7 pad 1: GND -> +5V
- U7 pad 2: unconnected-(U7-Pad2) -> GND
- U7 pad 3: (no net) -> Net-(U7-EN)
- U7 pad 4: (no net) -> unconnected-(U7-NC-Pad4)
- U7 pad 5: (no net) -> +3.3V
Routing:
- net AD0: track 0.00 -> 86.9 mm, vias 0 -> 3
- net +12V: track 0.00 -> 78.6 mm, vias 0 -> 3
- net AD1: track 0.00 -> 77.6 mm, vias 0 -> 3
- net AD2: track 0.00 -> 76.8 mm, vias 0 -> 3
- net AD3: track 0.00 -> 73.6 mm, vias 0 -> 3
- net +3.3V: track 0.00 -> 73.4 mm, vias 0 -> 7
- net +5V: track 0.00 -> 67.3 mm, vias 0 -> 20
- net Decimal_Point: track 0.00 -> 52.7 mm, vias 0 -> 2
- net BCD_Lane1: track 0.00 -> 46.0 mm, vias 0 -> 2
- net BCD_Lane2: track 0.00 -> 43.2 mm, vias 0 -> 2
- net BCD_MuxA: track 0.00 -> 29.0 mm, vias 0 -> 3
- net Net-(U5-2A3): track 0.00 -> 26.9 mm, vias 0 -> 2
- net /Time2_Thousandths: track 0.00 -> 26.7 mm, vias 0 -> 2
- net BCD_MuxB: track 0.00 -> 26.7 mm, vias 0 -> 3
- net /Time2_Tens: track 0.00 -> 26.5 mm, vias 0 -> 2
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- added copper zone on In2.Cu, net +5V
- added copper zone on B.Cu, net GND
- added copper zone on F.Cu, net GND
- added copper zone on In1.Cu, net GND
Other:
- board outline added: 50.8 x 88.9 mm
- copper layers 2 -> 4
- board text added: "† Prairie Edge Cadets Finish Line Controller"
