File: hardware/finishBoard/FinishControllerBoard_v1.kicad_sch (KiCad schematic)
At the start: 23 parts, among them J1 Conn_01x04, J10 Comm, J11 Conn_01x02, J2 LCD_Top_Half, J3 LCD_Bottom_Half, J4 Time2, J5 Time1, J6 React1, J7 React2, J8 Analog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

Commit message: Finish Control Board completion for order
Parts:
- removed J10: Comm, Connector_JST:JST_EH_B3B-EH-A_1x03_P2.50mm_Vertical, symbol Connector_Generic:Conn_01x03
- removed J11: Conn_01x02, Connector_JST:JST_XH_B2B-XH-A_1x02_P2.50mm_Vertical, symbol Connector_Generic:Conn_01x02
- removed J2: LCD_Top_Half, Connector_JST:JST_VH_B8P-VH-B_1x08_P3.96mm_Vertical, symbol Connector_Generic:Conn_01x08
- removed J3: LCD_Bottom_Half, Connector_JST:JST_VH_B8P-VH-B_1x08_P3.96mm_Vertical, symbol Connector_Generic:Conn_01x08
- removed J6: React1, Connector_JST:JST_VH_B10P-VH-B_1x10_P3.96mm_Vertical, symbol Connector_Generic:Conn_01x10
- removed J7: React2, Connector_JST:JST_VH_B10P-VH-B_1x10_P3.96mm_Vertical, symbol Connector_Generic:Conn_01x10
- added C3: 0.1uF, Capacitor_SMD:C_0805_2012Metric, symbol Device:C
- added J2: Comm, Connector_JST:JST_EH_B3B-EH-A_1x03_P2.50mm_Vertical, symbol Connector_Generic:Conn_01x03
- added J3: 12V Pwr, Connector_Molex:Molex_Nano-Fit_105309-xx02_1x02_P2.50mm_Vertical, symbol Connector_Generic:Conn_01x02
- added J6: Dsply Pwr, Connector_Molex:Molex_Nano-Fit_105309-xx04_1x04_P2.50mm_Vertical, symbol Connector_Generic:Conn_01x04
- added R23, R24, R25, R26: 100, Resistor_SMD:R_0805_2012Metric, symbol Device:R
- added U5: 74HCT244, Package_SO:SOIC-20W_7.5x12.8mm_P1.27mm, symbol 74xx:74HCT244
- H1, H2, H3, H4: footprint MountingHole:MountingHole_3.2mm_M3_Pad_TopBottom -> MountingHole:MountingHole_2.5mm_Pad
- J1: value Conn_01x04 -> Sensors
- J4, J5: footprint Connector_JST:JST_VH_B10P-VH-B_1x10_P3.96mm_Vertical -> Connector_JST:JST_EH_B10B-EH-A_1x10_P2.50mm_Vertical
- R5: value 22 -> 100
- R6: value 12k -> 100
- R7: value 1k -> 100
Connections:
- net LCD Right Latching/Time2_Hundredths Latched is gone; now on net Time2_Hundredths: J4.9 (Pin_9)
- net LCD Right Latching/Time2_Ones Latched is gone; now on net Time2_Ones: J4.7 (Pin_7)
- net LCD Right Latching/Time2_Tens Latched is gone; now on net Time2_Tens: J4.6 (Pin_6)
- net LCD Right Latching/Time2_Tenths Latched is gone; now on net Time2_Tenths: J4.8 (Pin_8)
- net LCD Right Latching/Time2_Thousandths Latched is gone; now on net Time2_Thousandths: J4.10 (Pin_10)
- net LCD_RS/CS is gone; now on net D8: R8.2
- net Time2_Decimal_Point is gone; now on net Decimal_Point: J4.5 (Pin_5)
- net *D3: now also R25.2
- net *D9: now also R7.2; no longer R19.2
- net +12V: now also J6.1 (Pin_1)
- net +5V: now also C3.1, J6.4 (Pin_4), U5.20 (VCC); no longer R5.2, R6.2
- net A2: now also R5.1
- net A3: now also R6.1
- net AD0: now also U5.12 (1Y3)
- net AD1: now also U5.3 (2Y0)
- net AD2: now also U5.5 (2Y1)
- net AD3: now also U5.7 (2Y2)
- net BCD_Lane1: now also R5.2
- net BCD_Lane2: now also R6.2
- net BCD_MuxA: now also U5.18 (1Y0)
- net BCD_MuxB: now also U5.16 (1Y1)
- net BCD_MuxC: now also U5.14 (1Y2)
- net D2: now also R26.2
- net D7: now also R18.2; no longer R8.1
- net D8: no longer R18.2
- net GND: now also C3.2, J2.3 (Pin_3), J6.2 (Pin_2), J6.3 (Pin_3), U5.1 (1OE), U5.10 (GND), U5.19 (2OE); no longer R7.1
- net Logic Level Shifter/Rx_HV_Out: now also J2.2 (Pin_2)
- net Logic Level Shifter/Tx_HV_In: now also J2.1 (Pin_1)
- net PowerManagement/+12Vsrc: now also J3.1 (Pin_1)
- net PowerManagement/GNDsrc: now also J3.2 (Pin_2)
- net Clock1 renamed *D5
- net *D5: now also R23.2
- net Clock2 renamed A6
- net LCD_E: no longer names the net of R19.1
- net LCD_E: now also U5.17 (2A0)
- net LCD_R/NW: no longer names the net of R18.1
- net LCD_R/NW: now also U5.15 (2A1)
- net Latch1 renamed D4
- net D4: now also R24.2
- net Latch2 renamed A7
- net Ser1 renamed *D6
- net *D6: now also R19.2
- net Ser2 renamed A5/SCL
- net Time1_Decimal_Point renamed Decimal_Point
- net Decimal_Point: now also U5.9 (2Y3)
- new net: R8.1, U5.13 (2A2)
- new net: R26.1, U5.2 (1A0)
- new net: R23.1, U5.8 (1A3)
- new net: R7.1, U5.11 (2A3)
- new net: R25.1, U5.4 (1A1)
- new net: R24.1, U5.6 (1A2)
Other:
- sheet Digit Demux Left renamed Digit Demux
- removed sheet Digit Demux Right
- removed sheet IO Expander
- removed sheet LCD Left Latching
- removed sheet LCD Right Latching
- sheet Digit Demux: file Digit_Demux_L.kicad_sch -> Digit_Demux.kicad_sch
- sheet Digit Demux ports: added BCD_Lane2, Time1_Hundredths Latched, Time1_Ones Latched, Time1_Tens Latched, Time1_Tenths Latched, Time1_Thousandths Latched, Time2_Hundredths Latched, Time2_Ones Latched, Time2_Tens Latched, Time2_Tenths Latched, Time2_Thousandths Latched; removed BCD_React, BCD_Time, React1_Hundredths, React1_Ones, React1_Tens, React1_Tenths, React1_Thousandths, Time1_Hundredths, Time1_Ones, Time1_Tens, Time1_Tenths, Time1_Thousandths
- sheet FinishSensors ports: added +3.3V, +5V, GND; removed none
- sheet PowerManagement ports: added +33Vcc; removed none
- note removed: "Multiple 74HC137 Demultiplexers: Schematic shows separate demux for each display (U12, U16, U17) Could use ONE demux with proper addressing scheme Current design wastes 2 ICs"
- note removed: "Shift Register Usage: Two 74HC595s provide 16 outputs Many outputs appear unused (bits 5-7 of lower byte) Could optimize bit allocation"
- note removed: "use 100 ohm across the board to any micro pins"
- moved on the sheet: J1, J4, J8, J9, R12, R13
